File: hardware/sensor-board/sensor-board.kicad_sch (KiCad schematic)
At the start: 83 parts, among them J1 HELM, J2 TACH, J3 PROBES, J4 RPi GPIO, J5 NMEA 2000, J6 LIGHTS, J7 5V IN, Q1 IRLML0030, U1 ADS1115IDGSR, U2 ADS1115IDGSR, U3 EL817, U4 MCP2518FD, U5 ISO1044BD, U6 UA78L05, U7 LM74700-Q1, Y1 40MHz

Commit message: Sensor board: no probe input; J6 gets its own I2C bus
No temperature probes on this boat: engine temperature comes from the temp
gauge's sender (J1 TEMP), water temperature from the depth transducer on
NMEA 2000. J3 and its 1-Wire parts (D8, R24, R25, GPIO26) are gone.

J6 moves to J3's old spot on the right edge, next to the header pins it
uses, and its SDA/SCL leave the converters' bus for a bus of their own:
i2c-gpio on GPIO5/6 (dtoverlay=i2c-gpio,bus=7,...; BOAT_LED_I2C_BUS=7),
4.7k pull-ups on the board (R24, R25). A stuck or shorted LED board can't
stall the engine data, and a bit-banged bus handles clock stretching,
which a microcontroller on the LED board may do and the Pi's hardware I2C
gets wrong. No hardware I2C pair is free at that corner of the header.

Routing: other nets now stay out of the half-pitch square round each of
the header's GND pins, on both layers. Tracks squeezed past them kept
starving their thermal spokes (pins 6, 14, 20, 25, 30, 34, 39 in turn);
this ends it for good.

SENSOR_BOARD.md says what J6 is enough for: PCA9685s at 16 PWM channels
each (four RGBW strips per chip, up to 62 chips), two independent
addressable data lines, and an RP2040 on the LED board for more.
The LED PWM driver opens BOAT_LED_I2C_BUS (defaults to BOAT_I2C_BUS).
Calibration page hides the probe card on the sensor board unless one
appears.

541 tests pass. ERC, DRC and parity: clean.

Co-Authored-By: Claude Opus 5.5 <noreply@anthropic.com>
Parts:
- removed D8: SMAJ5.0A, Diode_SMD:D_SMA, symbol Diode:SMAJ5.0A
- removed J3: PROBES, Connector_Phoenix_MC:PhoenixContact_MC_1,5_3-GF-3.81_1x03_P3.81mm_Horizontal_ThreadedFlange, symbol Connector_Generic:Conn_01x03
- J6: Note to the LED board: 1 3V3 (logic only, under 50 mA), 2 SDA, 3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 -> to the LED board: 1 3V3 (logic only, under 50 mA), 2 SDA GP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
- R24: Note 1-Wire pull-up -> J6 I2C pull-up (SDA, GPIO5)
- R25: value 100 -> 4.7k; MPN RC0805FR-07100RL -> RC0805FR-074K7L; Note 1-Wire series resistor -> J6 I2C pull-up (SCL, GPIO6)
Connections:
- net OW_EXT is gone; now on net LIGHT_SCL: R25.1
- net +3V3: now also R25.2
- net SCL: no longer J6.3 (Pin_3)
- net SDA: no longer J6.2 (Pin_2)
- net LIGHT_SDA: now reaches J4.29 (Pin_29)
- net LIGHT_SDA: now also J6.2 (Pin_2), R24.1
- net LIGHT_SCL: now reaches J4.31 (Pin_31)
- net LIGHT_SCL: now also J6.3 (Pin_3)
- removed net OW: J4.37 (Pin_37), R24.1, R25.2
- no-connect marks 25 -> 24
Other:
- note added: "J6 carries logic only: the strips' 12 V and current stay on the LED board. PWM strips: PCA9685s on the LED board's own I2C bus, GPIO5/6 (dtoverlay=i2c-gpio,bus=7,i2c_gpio_sda=5,i2c_gpio_scl=6). Addressable strips: DAT1 = GPIO18 (PWM0), DAT2 = GPIO19 (PWM1), 3.3 V: buffer to 5 V there. AUX = GPIO21, spare. 3V3 for the LED board's logic, under 50 mA."
- note removed: "1-WIRE PROBES"
- note removed: "J6 carries logic only: the strips' 12 V and current stay on the LED board. PWM strips: PCA9685s on SDA/SCL (not 0x48/0x49, the converters, or 0x70). Addressable strips: DAT1 = GPIO18 (PWM0), DAT2 = GPIO19 (PWM1), 3.3 V: buffer to 5 V there. AUX = GPIO21, spare. 3V3 for the LED board's logic, under 50 mA."
- note removed: "TEMPERATURE PROBES"
- moved on the sheet: R24, R25

Commit message: Sensor board: tap resistors all on the board, plain wire to the gauges
Each tap's top resistor is now a single 49.9k 1% 1206 on the board
(R1, R2, R4-R6), in place of 39k here plus a 10k soldered into the tap
wire at the gauge end. The tap wires are plain wire from the gauge
terminals to J1; nothing to solder into the harness.

The trade-off, at the owner's call: a tap wire is now part of its gauge's
circuit, so one chafed to ground would read like a shorted sender on that
gauge (and on IGN would short the key-on 12 V). SENSOR_BOARD.md says so
and says to route and secure them accordingly.

BOAT_TAP_R_TOP defaults to 49900 (49000 for a rev 1.0-1.1 board). The
tap levels are ratios, so the setting only moves the gauge-supply volts.
Legend, schematic notes, BOM, wiring steps, bring-up and order sheet
updated; the gauge-end resistors are off the shopping list.

541 tests pass. ERC, DRC and parity: clean.

Co-Authored-By: Claude Opus 5.5 <noreply@anthropic.com>
Parts:
- R1, R2, R4, R5, R6: value 39k -> 49.9k; MPN RC1206FR-0739KL -> RC1206FR-0749K9L
Other:
- note added: "Each gauge tap: the S (or I) terminal -> tap wire -> J1 -> 49.9k -> node (10k to GND, BAT54S clamp to GND/3V3) -> 1k -> ADC, with 100n at the ADC pin. V_adc = V_tap x 10/59.9 (0-16 V -> 0-2.7 V). Battery: 47k, x 10/57. Tach, Delco EST coil (BAT +12 V in, TACH out): J2-1 to the gray wire from the coil's TACH terminal, J2-2 to the tach gauge's G. The tach stays connected. TACH is the coil's switche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"
- note removed: "Each gauge tap: the S (or I) terminal -> 10k in heatshrink AT THE GAUGE -> J1 -> 39k -> node (10k to GND, BAT54S clamp to GND/3V3) -> 1k -> ADC, with 100n at the ADC pin. V_adc = V_tap x 10/59 (0-16 V -> 0-2.7 V). Battery: 47k on board, no remote resistor, x 10/57. Tach, Delco EST coil (BAT +12 V in, TACH out): J2-1 to the gray wire from the coil's TACH terminal, J2-2 to the tach gauge's G. The t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"
