File: hardware/sensor-board/sensor-board.kicad_sch (KiCad schematic)
At the start: 81 parts, among them J1 HELM, J2 TACH, J4 RPi GPIO, J5 NMEA 2000, J6 LIGHTS, J7 5V IN, Q1 IRLML0030, U1 ADS1115IDGSR, U2 ADS1115IDGSR, U3 EL817, U4 MCP2518FD, U5 ISO1044BD, U6 UA78L05, U7 LM74700-Q1, Y1 40MHz

Commit message: Sensor board rev 1.3: the LED link is an RJ45; LED board routing progress
Sensor board:
- J6 (JST GH) becomes an RJ45 on a new tab above the Pi's GPIO edge,
  facing up, with a PCA9615 (U8) carrying the LED board's I2C bus
  (GPIO5/6) as differential I2C over a straight-through patch cable, and
  each pair terminated 620/120/620 at 5 V. GPIO 18, 19 and 21 are freed:
  the LED board's RP2040 makes the addressable data itself now.
- board.py gains the LED board's dry run (padgeom.py: placement and
  routing without KiCad, checked for unrouted nets and overlaps); the
  whole board routes in it. KiCad's paths are in kicadpaths.py.

LED board:
- The RP2040's pins are fanned out before routing -- signals outward,
  supplies inward to vias under the chip -- and its I2C moves to GPIO4/5
  (pixel data on GPIO0-3) so neither crosses the other; the firmware
  follows. The link's SDA pair routes before SCL. Its corner now routes
  completely; a few long nets elsewhere are still open.

Co-Authored-By: Claude Opus 5.5 <noreply@anthropic.com>
Claude-Session: https://claude.ai/code/session_01VGxUaRe1pLvK1HEem77SSs
Parts:
- added C22, C23: 100n, sensor-board:C_0805_2012Metric_NoSilk, symbol Device:C
- added R29, R31, R32, R34: 620, sensor-board:R_0805_2012Metric_NoSilk, symbol Device:R
- added R30, R33: 120, sensor-board:R_0805_2012Metric_NoSilk, symbol Device:R
- added U8: PCA9615DP, Package_SO:TSSOP-10_3x3mm_P0.5mm, symbol Interface:PCA9615DP
- J6: footprint Connector_JST:JST_GH_SM08B-GHS-TB_1x08-1MP_P1.25mm_Horizontal -> Connector_RJ:RJ45_Amphenol_54602-x08_Horizontal; symbol Connector_Generic:Conn_01x08 -> Connector:RJ45; MPN SM08B-GHS-TB(LF)(SN); plug GHR-08V-S (JST GH, 1.25 mm, latc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 -> Amphenol 54602-908LF; Note to the LED board: 1 3V3 (logic only, under 50 mA), 2 SDA GP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 -> to the LED board's J1: a straight-through Cat5e/Cat6 patch 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
- R24: Note J6 I2C pull-up (SDA, GPIO5) -> LED board I2C pull-up (SDA, GPIO5)
- R25: Note J6 I2C pull-up (SCL, GPIO6) -> LED board I2C pull-up (SCL, GPIO6)
Connections:
- net +3V3: now also C22.1, U8.1 (V_{DD(A)}), U8.3 (EN); no longer J6.1 (Pin_1)
- net +5V: now also C23.1, R29.1, R32.1, U8.10 (V_{DD(B)})
- net GND: now also C22.2, C23.2, R31.2, R34.2, U8.5 (V_{SS}); no longer J6.4 (Pin_4), J6.7 (Pin_7)
- net LIGHT_SCL: now also U8.4 (SCL); no longer J6.3 (Pin_3)
- net LIGHT_SDA: now also U8.2 (SDA); no longer J6.2 (Pin_2)
- net LIGHT_AUX: no longer names the net of J6.8
- net LIGHT_AUX: no longer J4.40 (Pin_40)
- net LIGHT_DAT1: no longer names the net of J6.5
- net LIGHT_DAT1: no longer J4.12 (Pin_12)
- net LIGHT_DAT2: no longer names the net of J4.35 (Pin_35)
- net LIGHT_DAT2: no longer J6.6 (Pin_6)
- new net LINK_SCLM: J6.1, R30.2, R31.1, U8.6 (DSCLM)
- new net LINK_SCLP: J6.2, R29.2, R30.1, U8.7 (DSCLP)
- new net LINK_SDAM: J6.6, R33.2, R34.1, U8.9 (DSDAM)
- new net LINK_SDAP: J6.3, R32.2, R33.1, U8.8 (DSDAP)
- no-connect marks 24 -> 31
Other:
- note added: "J6: a straight-through Cat5e/Cat6 patch cable to the LED board's J1 -- NOT Ethernet: never into a switch or PoE. The LED board's own I2C bus, GPIO5/6 (dtoverlay=i2c-gpio,bus=7,i2c_gpio_sda=5,i2c_gpio_scl=6), as differential I2C: pairs 1/2 SCL, 3/6 SDA, each 620/120/620 at both ends; 4/5 and 7/8 reserved. No ground or power in the cable. On it: the LED board's PCA9685 (0x40), INA226 (0x45) and RP2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"
- note added: "LIGHTS: the RJ45 link to the LED board (differential I2C)"
- note removed: "J6 carries logic only: the strips' 12 V and current stay on the LED board. PWM strips: PCA9685s on the LED board's own I2C bus, GPIO5/6 (dtoverlay=i2c-gpio,bus=7,i2c_gpio_sda=5,i2c_gpio_scl=6). Addressable strips: DAT1 = GPIO18 (PWM0), DAT2 = GPIO19 (PWM1), 3.3 V: buffer to 5 V there. AUX = GPIO21, spare. 3V3 for the LED board's logic, under 50 mA."
- note removed: "LIGHTS: to a separate LED board"
- moved on the sheet: R24, R25

Commit message: Sensor board rev 1.3 built and checked, with a house battery input; the dashboard reads it
The boat has two batteries on a common negative, positives kept apart (house: lights and
stereo). J1.8, a second GND until now, becomes HSE+: the house battery through the same
47k/10k divider, BAT54S clamp and 1k/100n filter as the engine battery (J1.3, now labelled
ENG+), into U2 AIN2 (software channel 6). Its parts (R35-R37, D13, C24) take the next free
numbers; with no room left in the input column, its lane runs right to left beside U2.
design.channel_refs/channel_sch give each channel its parts and its place on the schematic.

Rev 1.3 (the cloud session's RJ45 link) is now built under KiCad and passes ERC, DRC and
parity with nothing reported; fab/ is regenerated from it. Fixes on the way: the RJ45's two
labels moved off the link's resistors and the board edge into the strip left of the jack
("J6 LED LINK", "NOT ETHERNET"); C22's GND pad, boxed in with room for one thermal spoke,
joins GND by its own via rather than the top pour; the legend moves down 1 mm for the new lane.

Dashboard: BOAT_HOUSE_BATTERY=true reads it (in tap and n2k modes). The BATTERY tile shows
"HOUSE 13.2 V" under its label, level with the engine battery's number (fits at 1180, 1280
and 1920 wide); house low/high alarms in the battery tile's menu, shown only where there is a
house reading, without painting the engine battery's bar; its own calibration on /calibrate;
a "House battery" data box; the simulator has a house battery charged while the engine runs.

Co-Authored-By: Claude Opus 5.5 <noreply@anthropic.com>
Parts:
- added C24: 100n, sensor-board:C_0805_2012Metric_NoSilk, symbol Device:C
- added D13: BAT54S, sensor-board:SOT-23_NoSilk, symbol Diode:BAT54S
- added R35: 47k, sensor-board:R_1206_3216Metric_NoSilk, symbol Device:R
- added R36: 10k, sensor-board:R_0805_2012Metric_NoSilk, symbol Device:R
- added R37: 1k, sensor-board:R_0805_2012Metric_NoSilk, symbol Device:R
- C22, C23: footprint sensor-board:C_0805_2012Metric_NoSilk -> sensor-board:C_0402_1005Metric_NoSilk; MPN CL21B104KBCNNNC -> CL05B104KO5NNNC
- J1: Note FUEL/TRIM/OIL/TEMP: that gauge's S terminal; BAT+: the dash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 -> FUEL/TRIM/OIL/TEMP: that gauge's S terminal; ENG+ / HSE+: t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
- R29, R31, R32, R34: footprint sensor-board:R_0805_2012Metric_NoSilk -> sensor-board:R_0402_1005Metric_NoSilk; MPN RC0805FR-07620RL -> RC0402FR-07620RL
- R30, R33: footprint sensor-board:R_0805_2012Metric_NoSilk -> sensor-board:R_0402_1005Metric_NoSilk; MPN RC0805FR-07120RL -> RC0402FR-07120RL
- U2: Note I2C 0x49: oil, engine temperature -> I2C 0x49: oil, engine temperature, house battery
Connections:
- net +3V3: now also D13.2 (K)
- net GND: now also C24.2, D13.1 (A), R36.2; no longer J1.8 (Pin_8)
- net HOUSE_ADC: now reaches U2.6 (AIN2)
- net HOUSE_ADC: now also C24.1, R37.2
- new net HOUSE_DIV: D13.3 (COM), R35.2, R36.1, R37.1
- new net HOUSE_IN: J1.8 (Pin_8), R35.1
- no-connect marks 31 -> 30
Other:
- note added: "HOUSE: J1.8 -> U2 AIN2"
